File: electric_pass_baseboard.kicad_pcb (KiCad board)
At the start: 2 copper layers, 50 x 100 mm, 147 parts, among them J1 USB_C_Receptacle_USB2.0_16P, J2 Conn_02x05_Counter_Clockwise, J3 Conn_02x05_Counter_Clockwise, Q1 AO3401A, SW1 MSK12C02, SW2 TS24CA, SW4 TS24CA, SW5 TS24CA, SW6 TS24CA, SW9 TS24CA, U1 TP4056-42-ESOP8, U2 EA3036C, U3 F1C200S, U4 FPC 0.5mm 40P 下接, U5 FPC 0.5mm 40P 上接, U6 W25N01GVZEIG_C907680, U7 LSM6DS3, U8 WAFER-MX1.25-2PWB, U9 STI9287C, Y1 24Mhz 12pF

Commit message: V0.5
Parts:
- removed C38, C39: 100nF, Capacitor_SMD:C_0603_1608Metric
- removed the G*** at (159.7, 69.8)
- removed R3, R4, R43, R49: 10K, Resistor_SMD:R_0603_1608Metric
- removed R47, R48: 0R, Resistor_SMD:R_0603_1608Metric
- removed U7: LSM6DS3, Package_LGA:LGA-14_3x2.5mm_P0.5mm_LayoutBorder3x4y
- added C46: 100nF, Capacitor_SMD:C_0603_1608Metric, F.Cu at (161.8, 122.4)
- added C47: 100nF, Capacitor_SMD:C_0603_1608Metric, F.Cu at (132.0, 127.5)
- added C48: 10uF, Capacitor_SMD:C_0603_1608Metric, F.Cu at (163.3, 119.3)
- added F1: Fuse, Fuse:Fuse_0805_2012Metric, F.Cu at (145.5, 137.8)
- added G***: LOGO, shirogane:prts_simp, B.Cu at (160.1, 69.8)
- added Q2: AO3401A, Package_TO_SOT_SMD:SOT-23, F.Cu at (134.1, 124.3)
- added R32: 10K, Resistor_SMD:R_0603_1608Metric, F.Cu at (163.3, 107.8)
- added TP12: TestPoint, TestPoint:TestPoint_Pad_D1.0mm, F.Cu at (143.6, 127.4)
- added U10: ZX-SH1.0-2PWT, EasyEDA:CONN-SMD_2P-P1.00_HX-1.0-2P-WT, F.Cu at (149.5, 134.8)
- C35: value 10uF -> 1uF
- D2, D5: value 1N5819 SS14 -> 1N5819WS
- FID1, FID2, FID4: footprint Fiducial:Fiducial_1mm_Mask2mm -> Fiducial:Fiducial_1mm_Mask3mm
- FID3: footprint Fiducial:Fiducial_1mm_Mask2mm -> shirogane:Fiducial_1mm_Mask3mm
- R13: value 2K -> 5.1K
- R40: value 0R -> 10R
- SW1: value MSK12C02 -> TS24CA; footprint EasyEDA:SW-TH_MSK12C02 -> EasyEDA:SW-SMD_TS24CA
- TP1, TP10, TP11, TP2, TP3, TP4, TP5, TP6, TP7, TP8, TP9: footprint TestPoint:TestPoint_Pad_D1.5mm -> TestPoint:TestPoint_Pad_D1.0mm
- U4: value FPC 0.5mm 40P 下接 -> 3寸液晶屏TFT 全新无定义资料
- U5: value FPC 0.5mm 40P 上接 -> ST7701 IPS; footprint Connector_FFC-FPC:Hirose_FH12-40S-0.5SH_1x40-1MP_P0.50mm_Horizontal -> shirogane:FPC-SMD_40P-P0.50_HC-FPC-0.5-40P-CSH20
- U8: value WAFER-MX1.25-2PWB -> GEK100-XX; footprint EasyEDA:CONN-SMD_2P-P1.25_XUNPU_WAFER-MX1.25-2PWB -> Package_TO_SOT_SMD:SOT-23-6
- moved FID3 176.0 mm to (1.77, 1.77)
- moved U8 14.4 mm to (134.9, 127.8), turned to 0 degrees
- moved R1 14.3 mm to (145.8, 136.1)
- moved R2 10.5 mm to (153.7, 128.0), turned to 90 degrees
- moved TP11 9.40 mm to (147.2, 128.9)
- moved R14 7.12 mm to (166.4, 126.3)
- moved FID4 7.08 mm to (168.0, 66.7)
- moved R40 7.03 mm to (158.8, 122.4)
- moved Q1 5.97 mm to (144.9, 133.3), turned to -90 degrees
- moved G*** 5.18 mm to (171.3, 121.5)
- moved R16 3.30 mm to (154.7, 110.4), turned to -90 degrees
- moved TP6 2.84 mm to (166.8, 100.3)
- moved D2 2.70 mm to (144.8, 130.4), turned to 0 degrees
- moved C30 2.40 mm to (164.7, 103.9), turned to 45 degrees
- moved TP3 2.13 mm to (166.4, 119.2)
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Connections:
- J1 pad A4: VBUS -> Net-(F1-Pad1)
- J1 pad A9: VBUS -> Net-(F1-Pad1)
- J1 pad B4: VBUS -> Net-(F1-Pad1)
- J1 pad B9: VBUS -> Net-(F1-Pad1)
- J2 pad 6: /PE11 -> /PE3
- R12 pad 1: VBAT_OUT -> +3.3V
- R14 pad 1: VBAT_OUT -> GND
- R14 pad 2: Net-(U2-EN1) -> Net-(U1-PROG)
- SW1 pad 1: VBAT_OUT -> GND
- SW1 pad 2: Net-(D2-K) -> GND
- SW1 pad 3: unconnected-(SW1-Pad3) -> GND
- SW1 pad 4: unconnected-(SW1-Pad4)_2 -> Net-(U8-KEY)
- SW2 pad 1: unconnected-(SW2-Pad1) -> GND
- SW2 pad 2: unconnected-(SW2-Pad2) -> GND
- SW4 pad 1: unconnected-(SW4-Pad1) -> GND
- SW4 pad 2: unconnected-(SW4-Pad2) -> GND
- SW5 pad 1: unconnected-(SW5-Pad1) -> GND
- SW5 pad 2: unconnected-(SW5-Pad2) -> GND
- SW6 pad 1: unconnected-(SW6-Pad1) -> GND
- SW6 pad 2: unconnected-(SW6-Pad2) -> GND
- SW9 pad 1: unconnected-(SW9-Pad1) -> GND
- SW9 pad 2: unconnected-(SW9-Pad2) -> GND
- U2 pad 18: Net-(U2-EN3) -> Net-(U2-EN1)
- U3 pad 38: /PE11 -> /screen/SCREEN_CS
- U3 pad 46: /screen/SCREEN_CS -> /PE3
- U3 pad 47: /soc_f1c/I2C_IRQ -> /power/PWR_SHUTDOWN
- U4 pad MP: (no net) -> GND
- U5 pad MP: (no net) -> GND
- U8 pad 3: GND -> Net-(U8-KEY)
- U8 pad 4: GND -> /power/PWR_SHUTDOWN
Routing:
- net /PE3: track 0.00 -> 62.0 mm, vias 0 -> 2
- net /PE11: track 57.4 -> 0.00 mm
- net /power/PWR_SHUTDOWN: track 0.00 -> 51.2 mm, vias 0 -> 2
- net /soc_f1c/I2C_IRQ: track 41.8 -> 0.00 mm, vias 4 -> 0
- net VBAT: track 35.4 -> 54.4 mm, vias 2 -> 4
- net +3.3V: track 300.5 -> 282.9 mm, vias 27 -> 24
- net Net-(J1-CC1): track 21.0 -> 4.51 mm
- net Net-(J1-CC2): track 2.07 -> 12.9 mm
- net Net-(U2-EN1): track 3.78 -> 14.2 mm, vias 0 -> 2
- net Net-(F1-Pad1): track 0.00 -> 9.13 mm
- net /VBAT_SENSE: track 50.6 -> 58.9 mm
- net Net-(Q2-G): track 0.00 -> 7.98 mm
- net VBUS: track 61.8 -> 54.2 mm, vias 0 -> 2
- net Net-(U8-KEY): track 0.00 -> 7.49 mm
- net /adc_periph/ADCBAT: track 11.8 -> 4.32 mm
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Other:
- board text added: "1- 2- 3- 4- FEL-"
- board text added: "Electronic Authorization Terminal 电子通行证终端 Model/型号: EPA-V04 Power/电源: 5V1A ACC ID: 3279ade LMIIT ID: 7355611 拉特兰机械制造总局受托制造"
- board text added: "GND SDA TVI TVO 3V3 SCL BSC AD2 AD3 AD4"
- board text added: "PWR"
- board text added: "Rhodes Island Electric Pass V0.5"
- board text added: "Rhodes Island Electronic Pass"
- board text added: "TF Card"
- board text added: "VBAT"
- board text added: "。"
- board text removed: "1"
- board text removed: "1 2 3 4 FEL"
- board text removed: "Electronic Authorization Terminal 电子通行证终端 Model/型号: EPA-V031 Power/电源: 5V1A ACC ID: 429a12 LMIIT ID: 7355608 拉特兰机械制造总局受托制造"
- board text removed: "GND SDA TVI TVO 3V3 SCL AD1 AD2 AD3 AD4"
- board text removed: "ON OFF"
- board text removed: "Rhodes Island Electric Pass"
- board text removed: "Rhodes Island Electric Pass V0.3.1"
