File: electric_pass_baseboard.kicad_pcb (KiCad board)
At the start: 4 copper layers, 50 x 100 mm, 154 parts, among them J1 USB_C_Receptacle_USB2.0_16P, J2 Conn_02x05_Counter_Clockwise, J3 Conn_02x05_Counter_Clockwise, Q1 AO3401A, Q2 AO3401A, SW1 TS24CA, SW2 TS24CA, SW4 TS24CA, SW5 TS24CA, SW6 TS24CA, SW9 TS24CA, U1 TP4056-42-ESOP8, U10 ZX-SH1.0-2PWT, U2 EA3036C, U3 F1C200S, U4 3寸液晶屏TFT 全新无定义资料, U5 ST7701 IPS, U6 W25N01GVZEIG_C907680, U7 PW1515, U8 GEK100-XX, U9 STI9287C, Y1 24Mhz 12pF

Commit message: added comment
Parts:
- moved U6 0.49 mm to (136.1, 102.9)
Routing:
- net /soc_peripherals/NAND_CLK: track 35.5 -> 36.6 mm
- net GND: track 145.1 -> 144.0 mm
- net +3.3V: track 304.4 -> 305.3 mm
- net /soc_f1c/SDIO_D1: track 54.9 -> 55.7 mm
- net /soc_f1c/SDIO_CMD: track 55.1 -> 55.9 mm
- net /soc_f1c/SDIO_D2: track 55.0 -> 55.8 mm
- net /soc_f1c/SDIO_D0: track 55.1 -> 55.9 mm
- net /soc_f1c/SDIO_D3: track 55.0 -> 55.7 mm
