File: btn_ladder.kicad_sch (KiCad schematic)
At the start: 12 parts, among them SW2 TS24CA, SW4 TS24CA, SW5 TS24CA, SW6 TS24CA

Commit message: added comment
Other:
- title: 明日方舟电子通行证 -> 明日方舟电子通行证F1C200s Ver
Changed lines of the file:
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@@
 	(paper "A4")
 	(title_block
-		(title "明日方舟电子通行证")
+		(title "明日方舟电子通行证F1C200s Ver")
 		(date "2025-11-26")
 		(rev "V0.3.1")
 		(company "Shirogane Tsumugi")
 		(comment 1 "V0.3 添加屏幕兼容接口，添加SD卡槽，优化布线")
-		(comment 2 "V0.3.1 BUG修复")
-		(comment 3 "V0.3.2（V0.4） 生产优化。")
-		(comment 4 "V0.5 实现按键开关机、低电量关机、拉出i2s")
+		(comment 2 "V0.4 生产优化")
+		(comment 3 "V0.5 实现按键开关机、低电量关机、拉出i2s")
+		(comment 4 "V0.6 添加OVPOCP、重做阻抗走四层板")
 	)
 	(text "ADC记得加电容哦 否则可能采样波动大\n感谢和光老师"
