File: electric_pass_baseboard.kicad_sch (KiCad schematic)
At the start: 22 parts, among them J1 USB_C_Receptacle_USB2.0_16P, J2 Conn_02x05_Counter_Clockwise, J3 Conn_02x05_Counter_Clockwise, U7 PW1515

Commit message: added comment
Other:
- title: 明日方舟电子通行证 -> 明日方舟电子通行证F1C200s Ver
- moved on the sheet: C38, D7, D8, J2, J3, R43, R45, Reference: R40, TP10, TP4, TP5, TP7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
