File: screen.kicad_sch (KiCad schematic)
At the start: 17 parts, among them U4 3寸液晶屏TFT 全新无定义资料, U5 ST7701 IPS, U9 STI9287C

Commit message: added comment
Other:
- note added: "Pin2Pin且兼容:SY7200A"
- note removed: "Alt.BOM:SY7200A"
- title: 明日方舟电子通行证 -> 明日方舟电子通行证F1C200s Ver
Changed lines of the file:
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@@
 	(paper "A4")
 	(title_block
-		(title "明日方舟电子通行证")
+		(title "明日方舟电子通行证F1C200s Ver")
 		(date "2025-11-26")
 		(rev "V0.3.1")
 		(company "Shirogane Tsumugi")
 		(comment 1 "V0.3 添加屏幕兼容接口，添加SD卡槽，优化布线")
-		(comment 2 "V0.3.1 BUG修复")
-		(comment 3 "V0.3.2（V0.4） 生产优化。")
-		(comment 4 "V0.5 实现按键开关机、低电量关机、拉出i2s")
+		(comment 2 "V0.4 生产优化")
+		(comment 3 "V0.5 实现按键开关机、低电量关机、拉出i2s")
+		(comment 4 "V0.6 添加OVPOCP、重做阻抗走四层板")
 	)
 	(text "*4/*5:开机默认背光状态\n贴R28: 默认开背光\n贴R7：默认关背光\n\n手动复刻建议贴R28 调试结束后贴R7\n批量直接R7+QC"
@@
 		)
 	)
-	(text "Alt.BOM:SY7200A"
+	(text "Pin2Pin且兼容:SY7200A"
 		(exclude_from_sim no)
 		(at 225.044 122.682 0)
