File: soc_peripherals.kicad_sch (KiCad schematic)
At the start: 10 parts, among them SW9 TS24CA, U6 W25N01GVZEIG_C907680

Commit message: added comment
Other:
- note added: "Pin2Pin且兼容： MX35LF1G GD5F1GQ4xA"
- title: 明日方舟电子通行证 -> 明日方舟电子通行证F1C200s Ver
Changed lines of the file:
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@@
 	(paper "A4")
 	(title_block
-		(title "明日方舟电子通行证")
+		(title "明日方舟电子通行证F1C200s Ver")
 		(date "2025-11-26")
 		(rev "V0.3.1")
 		(company "Shirogane Tsumugi")
 		(comment 1 "V0.3 添加屏幕兼容接口，添加SD卡槽，优化布线")
-		(comment 2 "V0.3.1 BUG修复")
-		(comment 3 "V0.3.2（V0.4） 生产优化。")
-		(comment 4 "V0.5 实现按键开关机、低电量关机、拉出i2s")
+		(comment 2 "V0.4 生产优化")
+		(comment 3 "V0.5 实现按键开关机、低电量关机、拉出i2s")
+		(comment 4 "V0.6 添加OVPOCP、重做阻抗走四层板")
+	)
+	(text "Pin2Pin且兼容：\nMX35LF1G\nGD5F1GQ4xA"
+		(exclude_from_sim no)
+		(at 84.074 111.76 0)
+		(effects
+			(font
+				(size 1.27 1.27)
+			)
+		)
 	)
 	(text "Force FEL Button"
